Commit message: Update wrist joint limits

File: urdf/valkyrie_sim.urdf (robot description, URDF)
Before this commit: robot valkyrie, 86 links, 85 joints
Links:
- removed link base_link
Joints:
- removed joint base_link_joint
- joint leftWristPitch: limit lower=-0.36 upper=0.49 effort=14 velocity=1 -> lower=-0.5 upper=0.5 effort=14 velocity=1
- joint leftWristRoll: limit lower=-0.62 upper=0.625 effort=14 velocity=1 -> lower=-0.2 upper=0.3 effort=14 velocity=1
- joint rightWristPitch: limit lower=-0.49 upper=0.36 effort=14 velocity=1 -> lower=-0.5 upper=0.5 effort=14 velocity=1
- joint rightWristRoll: limit lower=-0.625 upper=0.62 effort=14 velocity=1 -> lower=-0.2 upper=0.3 effort=14 velocity=1

File: urdf/valkyrie_sim_drake.urdf (robot description, URDF)
Before this commit: robot valkyrie, 84 links, 83 joints
Links:
- added link leftFootSole_Frame, mass 0
- added link rightFootSole_Frame, mass 0
Joints:
- added joint leftFootSole_Offset: type fixed, parent leftFoot, child leftFootSole_Frame, origin xyz=0.067  0 -0.09 rpy=0.0 0.0 0.0
- added joint rightFootSole_Offset: type fixed, parent rightFoot, child rightFootSole_Frame, origin xyz=0.067  0 -0.09 rpy=0.0 0.0 0.0
- joint leftWristPitch: limit lower=-0.36 upper=0.49 effort=14 velocity=1 -> lower=-0.5 upper=0.5 effort=14 velocity=1
- joint leftWristRoll: limit lower=-0.62 upper=0.625 effort=14 velocity=1 -> lower=-0.2 upper=0.3 effort=14 velocity=1
- joint rightWristPitch: limit lower=-0.49 upper=0.36 effort=14 velocity=1 -> lower=-0.5 upper=0.5 effort=14 velocity=1
- joint rightWristRoll: limit lower=-0.625 upper=0.62 effort=14 velocity=1 -> lower=-0.2 upper=0.3 effort=14 velocity=1
